File: _autosave-rigid.kicad_pcb (KiCad board)
At the start: 4 copper layers, 33 x 35 mm, 58 parts, among them J1 47219-2001, J2 Bus_PCI_Express_Mini, J3 Battery, J4 USB_C_Receptacle_USB2.0, J5 FH34SRJ-6S-0.5SH(50), J6 FH34SRJ-6S-0.5SH(50), J7 Conn_01x02_Female, U1 STM32L432KCUx, U2 BQ24072RGTT, U3 TPS63020DSJR, U4 AW9523BTQR, U5 ALC5672

Commit message: One piece board, a bit into PCB
Parts:
- moved J2 21.2 mm to (123.8, 74.3)
- moved J1 16.6 mm to (136.0, 90.6), turned to -90 degrees
- moved U1 13.4 mm to (126.5, 105.5)
Other:
- board size 33 x 35 mm -> 37.5 x 130 mm
Changed lines of the file:
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@@
   )
   (footprint "Package_DFN_QFN:QFN-32-1EP_5x5mm_P0.5mm_EP3.45x3.45mm" (layer "F.Cu")
-    (at 115 112.55)
+    (at 126.45 105.5)
     (descr "QFN, 32 Pin (http://www.analog.com/media/en/package-pcb-resources/package/pkg_pdf/ltc-legacy-qfn/QFN_32_05-08-1693.pdf), generated with kicad-footprint-generator ipc_noLead_generator.py")
     (tags "QFN NoLead")
@@
       (effects (font (size 0.64 0.64) (thickness 0.15)))
     )
-    (fp_text value "FH34SRJ-6S-0.5SH(50)" (at 7.2536 2.5436 90) (layer "F.Fab")
+    (fp_text value "FH34SRJ-6S-0.5SH(50)" (at -0.15 3.1 90) (layer "F.Fab")
       (effects (font (size 0.64 0.64) (thickness 0.15)))
     )
@@
   )
   (footprint "JLCPCB:MOLEX_67910-5700" (layer "F.Cu")
-    (at 123.85 95.45)
+    (at 123.75 74.3)
     (property "Sheetfile" "rigid.kicad_sch")
     (property "Sheetname" "")
@@
   )
   (footprint "JLCPCB:MOLEX_47219-2001" (layer "F.Cu")
-    (at 141.6 74.95 90)
+    (at 136 90.6 -90)
     (property "MANUFACTURER" "MOLEX")
     (property "Sheetfile" "rigid.kicad_sch")
@@
     (fp_line (start -6.8 5.9) (end -6.8 3.5) (layer "F.Fab") (width 0.127))
     (fp_line (start 6.8 -4.8) (end 6.8 5.9) (layer "F.Fab") (width 0.127))
-    (pad "1" smd rect locked (at 3.2 2.1 90) (size 0.8 1.5) (layers "F.Cu" "F.Paste" "F.Mask")
+    (pad "1" smd rect locked (at 3.2 2.1 270) (size 0.8 1.5) (layers "F.Cu" "F.Paste" "F.Mask")
       (net 22 "unconnected-(J1-Pad1)") (pinfunction "DAT2") (pintype "bidirectional+no_connect"))
-    (pad "2" smd rect locked (at 2.1 2.1 90) (size 0.8 1.5) (layers "F.Cu" "F.Paste" "F.Mask")
+    (pad "2" smd rect locked (at 2.1 2.1 270) (size 0.8 1.5) (layers "F.Cu" "F.Paste" "F.Mask")
       (net 23 "/~{CS_SD}") (pinfunction "CD/DAT3") (pintype "bidirectional"))
-    (pad "3" smd rect locked (at 1 2.1 90) (size 0.8 1.5) (layers "F.Cu" "F.Paste" "F.Mask")
+    (pad "3" smd rect locked (at 1 2.1 270) (size 0.8 1.5) (layers "F.Cu" "F.Paste" "F.Mask")
       (net 24 "/MOSI_SD") (pinfunction "CMD") (pintype "bidirectional"))
-    (pad "4" smd rect locked (at -0.1 2.1 90) (size 0.8 1.5) (layers "F.Cu" "F.Paste" "F.Mask")
+    (pad "4" smd rect locked (at -0.1 2.1 270) (size 0.8 1.5) (layers "F.Cu" "F.Paste" "F.Mask")
       (net 1 "+3V3") (pinfunction "VDD") (pintype "power_in"))
-    (pad "5" smd rect locked (at -1.2 2.1 90) (size 0.8 1.5) (layers "F.Cu" "F.Paste" "F.Mask")
+    (pad "5" smd rect locked (at -1.2 2.1 270) (size 0.8 1.5) (layers "F.Cu" "F.Paste" "F.Mask")
       (net 25 "/SCLK_SD") (pinfunction "CLK") (pintype "input"))
-    (pad "6" smd rect locked (at -2.3 2.1 90) (size 0.8 1.5) (layers "F.Cu" "F.Paste" "F.Mask")
+    (pad "6" smd rect locked (at -2.3 2.1 270) (size 0.8 1.5) (layers "F.Cu" "F.Paste" "F.Mask")
       (net 2 "GND") (pinfunction "VSS") (pintype "power_in"))
-    (pad "7" smd rect locked (at -3.4 2.1 90) (size 0.8 1.5) (layers "F.Cu" "F.Paste" "F.Mask")
+    (pad "7" smd rect locked (at -3.4 2.1 270) (size 0.8 1.5) (layers "F.Cu" "F.Paste" "F.Mask")
       (net 26 "/MISO_SD") (pinfunction "DAT0") (pintype "bidirectional"))
-    (pad "8" smd rect locked (at -4.5 2.1 90) (size 0.8 1.5) (layers "F.Cu" "F.Paste" "F.Mask")
+    (pad "8" smd rect locked (at -4.5 2.1 270) (size 0.8 1.5) (layers "F.Cu" "F.Paste" "F.Mask")
       (net 27 "unconnected-(J1-Pad8)") (pinfunction "DAT1") (pintype "bidirectional+no_connect"))
-    (pad "G1" smd rect locked (at 6.875 4.7 90) (size 1.5 2.05) (layers "F.Cu" "F.Paste" "F.Mask")
+    (pad "G1" smd rect locked (at 6.875 4.7 270) (size 1.5 2.05) (layers "F.Cu" "F.Paste" "F.Mask")
       (net 2 "GND") (pinfunction "GND@1") (pintype "power_in"))
-    (pad "G2" smd rect locked (at 6.875 -3.6 90) (size 1.5 2.05) (layers "F.Cu" "F.Paste" "F.Mask")
+    (pad "G2" smd rect locked (at 6.875 -3.6 270) (size 1.5 2.05) (layers "F.Cu" "F.Paste" "F.Mask")
       (net 2 "GND") (pinfunction "GND@2") (pintype "power_in"))
-    (pad "G3" smd rect locked (at -6.875 -3.6 90) (size 1.5 2.05) (layers "F.Cu" "F.Paste" "F.Mask")
+    (pad "G3" smd rect locked (at -6.875 -3.6 270) (size 1.5 2.05) (layers "F.Cu" "F.Paste" "F.Mask")
       (net 2 "GND") (pinfunction "GND@3") (pintype "power_in"))
-    (pad "G4" smd rect locked (at -6.875 4.7 90) (size 1.5 2.05) (layers "F.Cu" "F.Paste" "F.Mask")
+    (pad "G4" smd rect locked (at -6.875 4.7 270) (size 1.5 2.05) (layers "F.Cu" "F.Paste" "F.Mask")
       (net 2 "GND") (pinfunction "GND@4") (pintype "power_in"))
   )
   (gr_poly
     (pts
-      (xy 142 151)
-      (xy 109 151)
-      (xy 109 115.95)
-      (xy 142 115.95)
+      (xy 144.35 151)
+      (xy 106.8 151)
+      (xy 106.8 21)
+      (xy 144.35 21)
     ) (layer "Edge.Cuts") (width 0.1) (fill none))
+  (dimension (type aligned) (layer "F.Cu")
+    (pts (xy 106.75 155.3) (xy 144.25 155.35))
+    (height 3.35)
+    (gr_text "37.5000 mm" (at 125.497933 156.874999 359.9236057) (layer "F.Cu")
+      (effects (font (size 1.5 1.5) (thickness 0.3)))
+    )
+    (format (units 3) (units_format 1) (precision 4))
+    (style (thickness 0.2) (arrow_length 1.27) (text_position_mode 0) (extension_height 0.58642) (extension_offset 0.5) keep_text_aligned)
+  )
+  (dimension (type aligned) (layer "F.Cu")
+    (pts (xy 145.95 151) (xy 145.9 21))
+    (height 6.499961)
+    (gr_text "130.0000 mm" (at 154.224961 85.996808 -89.97796316) (layer "F.Cu")
+      (effects (font (size 1.5 1.5) (thickness 0.3)))
+    )
+    (format (units 3) (units_format 1) (precision 4))
+    (style (thickness 0.2) (arrow_length 1.27) (text_position_mode 0) (extension_height 0.58642) (extension_offset 0.5) keep_text_aligned)
+  )
   (segment (start 129.57 134.25) (end 129.76 134.25) (width 0.25) (layer "F.Cu") (net 2))
   (segment (start 127.76 132.44) (end 129.57 134.25) (width 0.25) (layer "F.Cu") (net 2))
