File: audio.kicad_sch (KiCad schematic)
At the start: 52 parts, among them J10 +, J11 -, J7 FH34SRJ-6S-0.5SH(50), J8 FH34SRJ-6S-0.5SH(50), J9 Conn_01x02_Female, U6 ALC5672

Commit message: New Audio
Parts:
- removed C18, C19, C20, C27: 22pF, Capacitor_SMD:C_0402_1005Metric, symbol Device:C
- removed C31: 4.7uF, Capacitor_SMD:C_0402_1005Metric, symbol Device:C
- removed C33: 10uF, Capacitor_SMD:C_0402_1005Metric, symbol Device:C_Polarized
- removed C35: 2.2uF, Capacitor_SMD:C_0402_1005Metric, symbol Device:C
- removed C47, C49: 4.7uF, Capacitor_SMD:C_0402_1005Metric, symbol Device:C_Polarized
- removed C48, C50: 100nF, Capacitor_SMD:C_0402_1005Metric, symbol Device:C
- removed J10: +, TestPoint:TestPoint_THTPad_2.0x2.0mm_Drill1.0mm, symbol Connector_Generic:Conn_01x01
- removed J11: -, TestPoint:TestPoint_THTPad_2.0x2.0mm_Drill1.0mm, symbol Connector_Generic:Conn_01x01
- removed J8: FH34SRJ-6S-0.5SH(50), lib_fp:HRS_FH34SRJ-6S-0.5SH(50), symbol JLCPCB:FH34SRJ-6S-0.5SH(50)
- removed J9: Conn_01x02_Female, Jumper:SolderJumper-2_P1.3mm_Open_Pad1.0x1.5mm, symbol Connector:Conn_01x02_Female
- removed LS2: Earphone, speakerpads:speakerpads, symbol Device:Earphone
- removed R26: 10k, Resistor_SMD:R_0402_1005Metric, symbol Device:R
- removed U6: ALC5672, lib_fp:ALC5672-VB-CGT_QFN-48_EP_6x6_Pitch0.4mm, symbol JLCPCB:ALC5672
- added C18, C31: 1uF 6.3V, symbol Device:C_Polarized
- added C19, C20: 0.1uF 6.3V, symbol Device:C_Polarized
- added C27, C35: 4.7uF 6.3V, symbol Device:C_Polarized
- added C33: 0.1uF 6.3V, Capacitor_SMD:C_0402_1005Metric, symbol Device:C
- added C47: 1uF X7R, Capacitor_SMD:C_0402_1005Metric, symbol Device:C
- added R18, R19: 10k, Resistor_SMD:R_0402_1005Metric, symbol Device:R
- added R30, R31: 33, Resistor_SMD:R_0603_1608Metric, symbol Device:R
- added U6: LM4889MMX/NOPB, lib_fp:LM4889MMX&slash_NOPB, symbol lib_sch:LM4889MMX{brace}slash}NOPB
- added U7: ALC5616-CGT, lib_fp:ALC5616-CGT, symbol lib_sch:ALC5616-CGT
- added U8: RT9193-18GB, lib_fp:RT9193-18GB, symbol lib_sch:RT9193-18GB
- C21, C24: value 22pF -> NC 22pF 6.3V; footprint Capacitor_SMD:C_0402_1005Metric -> Capacitor_SMD:C_0603_1608Metric
- C22, C23, C25: value 4.7uF -> NC 22pF 6.3V; footprint Capacitor_SMD:C_0402_1005Metric -> Capacitor_SMD:C_0603_1608Metric
- C26: value 10uF -> 0.1uF 6.3V
- C28: value 4.7uF -> 4.7uF 6.3V; footprint Capacitor_SMD:C_0402_1005Metric -> (none)
- C29: value 2.2uF -> 4.7uF 6.3V
- C30, C32, C34, C46: value 100nF -> 2.2uF 6.3V
- C36, C38: value 2.2uF -> 2.2uF 6.3V
- C37: value 2.2uF -> 1uF X7R
- C39, C40: value 1uF -> 0.1uF 6.3V
- C41: value 680pF -> 4.7uF 6.3V
- C42: value 680pF -> 2.2uF 6.3V
- C43: value 680pF -> 0.1uF 6.3V
- C44: value 680pF -> 22nF
- C45: value 2.2uF -> 0.1uF 6.3V
- LS1: now in the parts list
- R20, R21: value 0 -> 20k; footprint Resistor_SMD:R_0402_1005Metric -> Resistor_SMD:R_0603_1608Metric
- R22, R23: value 22 -> 20k; footprint Resistor_SMD:R_0402_1005Metric -> Resistor_SMD:R_0603_1608Metric; now left out of the parts list
- R24: value 1k -> 20k; footprint Resistor_SMD:R_0402_1005Metric -> Resistor_SMD:R_0603_1608Metric; now left out of the parts list
- R25: value 1k -> 47; footprint Resistor_SMD:R_0402_1005Metric -> Resistor_SMD:R_0603_1608Metric; now left out of the parts list
- R26: renamed from R30; footprint Resistor_SMD:R_0402_1005Metric -> Resistor_SMD:R_0603_1608Metric
- R27: value 10k -> 0; footprint Resistor_SMD:R_0402_1005Metric -> Resistor_SMD:R_0603_1608Metric; now left out of the parts list
- R28, R29: value 1k -> 22; footprint Resistor_SMD:R_0402_1005Metric -> Resistor_SMD:R_0603_1608Metric; now left out of the parts list
Connections:
- net +3V3: now also C37.2, C39.1, C41.2, R23.2, C31.1, U6.6 (VDD), U7.31 (MICVDD), U8.1 (VIN); no longer C29.2, C30.2, C34.2
- net DBVDD: now also R18.2, R19.2; no longer C45.2, C46.2, R27.2
- net GND: now also C21.2, C22.2, C23.1, C25.1, C37.1, C44.1, C46.2, C18.2, C31.2, C47.1, U6.7 (GND), U7.1 (JD1), U7.33 (CPGND/DGND), U8.2 (GND); no longer C21.1, C29.1, C30.1, C32.1, C34.1, C41.2, C43.1, C43.2, C44.2, C46.1
- net GNDA: now also C29.1, C34.1, C36.1, C39.2, C41.1, R28.1, R29.1, C27.2, C33.2, C35.2, U7.18 (CPVREF), U7.7 (AGND); no longer C22.1, C23.2, C25.1, C37.1
- net OUT2+: now also U7.3 (IN2P)
- net OUT2-: now also U7.4 (IN2N/JD2)
- net PCM_CLOCK: now also C22.1, U7.24 (BCLK1)
- net PCM_DIN: now also C23.2, U7.21 (ADCDAT1)
- net PCM_DOUT: now also C21.1, U7.22 (DACDAT1)
- net PCM_SYNC: now also C24.2, U7.23 (LRCK1)
- net SCL_CODEC: now also R19.1, U7.26 (SCL); no longer R27.1
- net SDA_CODEC: now also R18.1, U7.27 (SDA)
- net at R20.1: now also R22.2, U6.3 (+IN); no longer C22.2
- net at R20.2: now also C19.1
- net at C40.1: now also R31.2, U7.17 (HPO_R); no longer R23.2
- net at C40.2: now also R28.2
- net at R24.1: now also R21.1, U6.4 (-IN)
- net at LS1.1 (-), R24.2: now also U6.5 (VO1); no longer C44.1, R25.2
- net at R21.2: now also C20.1
- net +1V8: now reaches C26.1
- net +1V8: now also C45.2, C46.1, R25.1, C27.1, C33.1, C35.1, C47.2, U7.15 (CPVDD), U7.29 (DBVDD), U7.6 (AVDD), U8.5 (VOUT)
- net at C38.2: now also U7.19 (CPVEE)
- net at C36.2: now also U7.16 (CPVPP)
- net at R22.1: now also C18.1, U6.2 (BYPASS)
- net AMP_OFF: now reaches R23.1
- net AMP_OFF: now also U6.1 (~{SD})
- net at C32.2: now also U7.14 (CPP1)
- net at C42.1: now also U7.30 (DCVDD); no longer LS1.2 (+)
- net at C28.1: now also R25.2, U7.5 (DACREF)
- net MCLK: now reaches C25.2
- net MCLK: now also U7.25 (MCLK)
- new net: C43.1, R29.2
- new net: C30.1, U7.11 (CPN2)
- new net: C30.2, U7.12 (CPP2)
- new net: C32.1, U7.13 (CPN1)
- new net: C34.2, U7.2 (IN1P)
- new net: C43.2, R30.2, U7.20 (HPO_L)
- new net: R27.2, U7.32 (MICBIAS1)
- new net: C29.2, U7.8 (VREF)
- new net: LS1.2 (+), U6.8 (VO2)
- new net: C44.2, U8.4 (BP)
- new net 1V8_EN: U8.3 (EN)
- new net IN+: C19.2, U7.9 (LOUTL/P)
- new net IN-: C20.2, U7.10 (LOUTR/N)
Other:
- moved on the sheet: R26

Commit message: Getting There
Need to move keyboard down and finish routing to audio, then we're there!
Parts:
- removed U6: LM4889MMX/NOPB, lib_fp:LM4889MMX&slash_NOPB, symbol lib_sch:LM4889MMX{brace}slash}NOPB
- added U5: LM4889MM, lib_fp:LM4889MM, symbol lib_sch:LM4889MM
- C14: renamed from C18; footprint (none) -> Capacitor_SMD:C_0402_1005Metric
- C15: renamed from C19; value 0.1uF 6.3V -> 100nF 6.3V; footprint (none) -> Capacitor_SMD:C_0402_1005Metric
- C16: renamed from C20; value 0.1uF 6.3V -> 100nF 6.3V; footprint (none) -> Capacitor_SMD:C_0402_1005Metric
- C22: renamed from C26; value 0.1uF 6.3V -> 100nF 6.3V
- C23: renamed from C27; footprint (none) -> Capacitor_SMD:C_0402_1005Metric
- C24: renamed from C31; footprint (none) -> Capacitor_SMD:C_0402_1005Metric
- C25: renamed from C28; footprint (none) -> Capacitor_SMD:C_0402_1005Metric
- C29: renamed from C33; value 0.1uF 6.3V -> 100nF 6.3V
- C31: renamed from C35; footprint (none) -> Capacitor_SMD:C_0402_1005Metric
- C35: renamed from C39; value 0.1uF 6.3V -> 100nF 6.3V
- C36: renamed from C40; value 0.1uF 6.3V -> 100nF 6.3V
- C39: renamed from C43; value 0.1uF 6.3V -> 100nF 6.3V
- C41: renamed from C45; value 0.1uF 6.3V -> 100nF 6.3V
- LS1: footprint (none) -> Connector_PinHeader_1.27mm:PinHeader_1x02_P1.27mm_Vertical
- U6: renamed from U7; MPN (none) -> C472693
- U7: renamed from U8; MPN (none) -> C27416
- renumbered C21 to C17, C22 to C18, C23 to C19, C24 to C20, C25 to C21, C29 to C26, C30 to C27, C32 to C28, C34 to C30, C36 to C32, C37 to C33, C38 to C34, C41 to C37, C42 to C38, C44 to C40, C46 to C42, C47 to C43, R20 to R19, R21 to R20, R22 to R21, R19 to R22
Connections:
- net +3V3: now also U5.6 (VDD)
- net AMP_OFF: now also U5.1 (~{SHDN})
- net GND: now also U5.7 (GND)
- net at R20.1, R24.1: now also U5.4 (-IN)
- net at LS1.1 (-), R24.2: now also U5.5 (VO1)
- net at C14.1, R21.1: now also U5.2 (BYPASS)
- net at R19.1, R21.2: now also U5.3 (+IN)
- net at LS1.2 (+): now also U5.8 (VO2)
Other:
- moved on the sheet: C14, C15, C16, C24, LS1, R19, R20, R21, R23, R24, R26

Commit message: First JLCPCB Ship!
Parts:
- removed R26: 0, Resistor_SMD:R_0603_1608Metric, symbol Device:R
- C22: renamed from C14; footprint Capacitor_SMD:C_0402_1005Metric -> Capacitor_SMD:C_0603_1608Metric; MPN (none) -> C15849
- C23: renamed from C15; footprint Capacitor_SMD:C_0402_1005Metric -> Capacitor_SMD:C_0603_1608Metric; MPN (none) -> C14663
- C24: renamed from C16; footprint Capacitor_SMD:C_0402_1005Metric -> Capacitor_SMD:C_0603_1608Metric; MPN (none) -> C14663
- C25: renamed from C17; now left out of the parts list
- C26: renamed from C18; now left out of the parts list
- C27: renamed from C19; now left out of the parts list
- C28: renamed from C20; now left out of the parts list
- C29: renamed from C21; now left out of the parts list
- C30: renamed from C22; MPN (none) -> C1525
- C31: renamed from C23; MPN (none) -> C23733
- C32: renamed from C24; footprint Capacitor_SMD:C_0402_1005Metric -> Capacitor_SMD:C_0603_1608Metric; MPN (none) -> C15849
- C33: renamed from C25; MPN (none) -> C23733
- C34: renamed from C26; MPN (none) -> C23733
- C35: renamed from C27; MPN (none) -> C12530
- C36: renamed from C28; MPN (none) -> C12530
- C37: renamed from C29; MPN (none) -> C1525
- C38: renamed from C30; MPN (none) -> C12530
- C39: renamed from C31; MPN (none) -> C23733
- C40: renamed from C32; MPN (none) -> C12530
- C41: renamed from C33; MPN (none) -> C52923
- C42: renamed from C34; MPN (none) -> C12530
- C43: renamed from C35; MPN (none) -> C1525
- C44: renamed from C36; MPN (none) -> C1525
- C45: renamed from C37; MPN (none) -> C23733
- C46: renamed from C38; MPN (none) -> C12530
- C47: renamed from C39; MPN (none) -> C1525
- C48: renamed from C40; MPN (none) -> C1532
- C49: renamed from C41; MPN (none) -> C1525
- C50: renamed from C42; MPN (none) -> C12530
- C51: renamed from C43; MPN (none) -> C52923
- LS1: now left out of the parts list
- R18, R22: MPN (none) -> C25744
- R19, R20, R21, R23, R24: MPN (none) -> C4184
- R25: M[N (none) -> C23182
- R27: renamed from R28; MPN (none) -> C23345
- R28: renamed from R29; M[N (none) -> C23345
- R29: renamed from R30; MPN (none) -> C23140
- R30: renamed from R31; MPN (none) -> C23140
- renumbered R27 to R26
Connections:
- net 1V8_EN is gone; now on net +3V3: U7.3 (EN)
- net DBVDD is gone; now on net +1V8: J7.2 (VDD), R18.2, R22.2
