File: keypad.kicad_sch (KiCad schematic)
At the start: 17 parts, among them SW10 3, SW11 6, SW12 9, SW13 #, SW14 End/Back, SW15 Up, SW16 Down, SW17 Call/OK, SW2 1, SW3 4, SW4 7, SW5 *, SW6 2, SW7 5, SW8 8, SW9 0, U5 AW9523BTQR

Commit message: Before Shortening
Parts:
- SW10, SW11, SW12, SW13, SW14, SW15, SW16, SW17, SW2, SW3, SW4, SW5, SW6, SW7, SW8, SW9: now left out of the parts list
Changed lines of the file:
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@@
   )
   (symbol (lib_id "Switch:SW_Push_45deg") (at 194.945 69.215 0) (unit 1)
-    (in_bom yes) (on_board yes) (fields_autoplaced)
+    (in_bom no) (on_board yes) (fields_autoplaced)
     (property "Reference" "SW15" (id 0) (at 194.945 60.96 0))
     (property "Value" "Up" (id 1) (at 194.945 63.5 0))
@@
   )
   (symbol (lib_id "Switch:SW_Push_45deg") (at 154.305 82.55 0) (unit 1)
-    (in_bom yes) (on_board yes) (fields_autoplaced)
+    (in_bom no) (on_board yes) (fields_autoplaced)
     (property "Reference" "SW8" (id 0) (at 154.305 74.295 0))
     (property "Value" "8" (id 1) (at 154.305 76.835 0))
@@
   )
   (symbol (lib_id "Switch:SW_Push_45deg") (at 194.945 97.155 0) (unit 1)
-    (in_bom yes) (on_board yes) (fields_autoplaced)
+    (in_bom no) (on_board yes) (fields_autoplaced)
     (property "Reference" "SW17" (id 0) (at 194.945 88.9 0))
     (property "Value" "Call/OK" (id 1) (at 194.945 91.44 0))
@@
   )
   (symbol (lib_id "Switch:SW_Push_45deg") (at 170.18 97.155 0) (unit 1)
-    (in_bom yes) (on_board yes) (fields_autoplaced)
+    (in_bom no) (on_board yes) (fields_autoplaced)
     (property "Reference" "SW13" (id 0) (at 170.18 88.9 0))
     (property "Value" "#" (id 1) (at 170.18 91.44 0))
@@
   )
   (symbol (lib_id "Switch:SW_Push_45deg") (at 138.43 82.55 0) (unit 1)
-    (in_bom yes) (on_board yes) (fields_autoplaced)
+    (in_bom no) (on_board yes) (fields_autoplaced)
     (property "Reference" "SW4" (id 0) (at 138.43 74.295 0))
     (property "Value" "7" (id 1) (at 138.43 76.835 0))
@@
   )
   (symbol (lib_id "Switch:SW_Push_45deg") (at 170.18 69.215 0) (unit 1)
-    (in_bom yes) (on_board yes) (fields_autoplaced)
+    (in_bom no) (on_board yes) (fields_autoplaced)
     (property "Reference" "SW11" (id 0) (at 170.18 60.96 0))
     (property "Value" "6" (id 1) (at 170.18 63.5 0))
@@
   )
   (symbol (lib_id "Switch:SW_Push_45deg") (at 138.43 69.215 0) (unit 1)
-    (in_bom yes) (on_board yes) (fields_autoplaced)
+    (in_bom no) (on_board yes) (fields_autoplaced)
     (property "Reference" "SW3" (id 0) (at 138.43 60.96 0))
     (property "Value" "4" (id 1) (at 138.43 63.5 0))
@@
   )
   (symbol (lib_id "Switch:SW_Push_45deg") (at 154.305 69.215 0) (unit 1)
-    (in_bom yes) (on_board yes) (fields_autoplaced)
+    (in_bom no) (on_board yes) (fields_autoplaced)
     (property "Reference" "SW7" (id 0) (at 154.305 60.96 0))
     (property "Value" "5" (id 1) (at 154.305 63.5 0))
@@
   )
   (symbol (lib_id "Switch:SW_Push_45deg") (at 170.18 82.55 0) (unit 1)
-    (in_bom yes) (on_board yes) (fields_autoplaced)
+    (in_bom no) (on_board yes) (fields_autoplaced)
     (property "Reference" "SW12" (id 0) (at 170.18 74.295 0))
     (property "Value" "9" (id 1) (at 170.18 76.835 0))
@@
   )
   (symbol (lib_id "Switch:SW_Push_45deg") (at 154.305 55.245 0) (unit 1)
-    (in_bom yes) (on_board yes) (fields_autoplaced)
+    (in_bom no) (on_board yes) (fields_autoplaced)
     (property "Reference" "SW6" (id 0) (at 154.305 46.99 0))
     (property "Value" "2" (id 1) (at 154.305 49.53 0))
@@
   )
   (symbol (lib_id "Switch:SW_Push_45deg") (at 138.43 55.245 0) (unit 1)
-    (in_bom yes) (on_board yes) (fields_autoplaced)
+    (in_bom no) (on_board yes) (fields_autoplaced)
     (property "Reference" "SW2" (id 0) (at 138.43 46.99 0))
     (property "Value" "1" (id 1) (at 138.43 49.53 0))
@@
   )
   (symbol (lib_id "Switch:SW_Push_45deg") (at 154.305 97.155 0) (unit 1)
-    (in_bom yes) (on_board yes) (fields_autoplaced)
+    (in_bom no) (on_board yes) (fields_autoplaced)
     (property "Reference" "SW9" (id 0) (at 154.305 88.9 0))
     (property "Value" "0" (id 1) (at 154.305 91.44 0))
@@
   )
   (symbol (lib_id "Switch:SW_Push_45deg") (at 194.945 82.55 0) (unit 1)
-    (in_bom yes) (on_board yes) (fields_autoplaced)
+    (in_bom no) (on_board yes) (fields_autoplaced)
     (property "Reference" "SW16" (id 0) (at 194.945 74.295 0))
     (property "Value" "Down" (id 1) (at 194.945 76.835 0))
@@
   )
   (symbol (lib_id "Switch:SW_Push_45deg") (at 170.18 55.245 0) (unit 1)
-    (in_bom yes) (on_board yes) (fields_autoplaced)
+    (in_bom no) (on_board yes) (fields_autoplaced)
     (property "Reference" "SW10" (id 0) (at 170.18 46.99 0))
     (property "Value" "3" (id 1) (at 170.18 49.53 0))
@@
   )
   (symbol (lib_id "Switch:SW_Push_45deg") (at 194.945 55.245 0) (unit 1)
-    (in_bom yes) (on_board yes) (fields_autoplaced)
+    (in_bom no) (on_board yes) (fields_autoplaced)
     (property "Reference" "SW14" (id 0) (at 194.945 46.99 0))
     (property "Value" "End/Back" (id 1) (at 194.945 49.53 0))
@@
   )
   (symbol (lib_id "Switch:SW_Push_45deg") (at 138.43 97.155 0) (unit 1)
-    (in_bom yes) (on_board yes) (fields_autoplaced)
+    (in_bom no) (on_board yes) (fields_autoplaced)
     (property "Reference" "SW5" (id 0) (at 138.43 88.9 0))
     (property "Value" "*" (id 1) (at 138.43 91.44 0))

Commit message: Getting There
Need to move keyboard down and finish routing to audio, then we're there!
Parts:
- added C13: 1uF, Capacitor_SMD:C_0603_1608Metric, symbol Device:C
- renumbered SW2 to SW1, SW11 to SW10, SW12 to SW11, SW13 to SW12, SW14 to SW13, SW15 to SW14, SW16 to SW15, SW17 to SW16, SW3 to SW2, SW4 to SW3, SW5 to SW4, SW6 to SW5, SW7 to SW6, SW8 to SW7, SW9 to SW8, SW10 to SW9, U5 to U4
Connections:
- net +3V3: now also C13.1
- net GND: now also C13.2
Changed lines of the file:
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@@
   (junction (at 172.72 99.695) (diameter 0) (color 0 0 0 0)
+  )
+  (junction (at 102.235 138.43) (diameter 0) (color 0 0 0 0)
   )
   (junction (at 172.72 85.09) (diameter 0) (color 0 0 0 0)
@@
   (symbol (lib_id "Switch:SW_Push_45deg") (at 194.945 69.215 0) (unit 1)
     (in_bom no) (on_board yes) (fields_autoplaced)
-    (property "Reference" "SW15" (id 0) (at 194.945 60.96 0))
+    (property "Reference" "SW14" (id 0) (at 194.945 60.96 0))
     (property "Value" "Up" (id 1) (at 194.945 63.5 0))
     (property "Footprint" "Keypad:snap dome" (id 2) (at 194.945 69.215 0)
@@
     (pin "2")
   )
+  (symbol (lib_id "Device:C") (at 102.235 142.24 0) (unit 1)
+    (in_bom yes) (on_board yes) (fields_autoplaced)
+    (property "Reference" "C13" (id 0) (at 105.41 140.9699 0)
+      (effects (font (size 1.27 1.27)) (justify left))
+    )
+    (property "Value" "1uF" (id 1) (at 105.41 143.5099 0)
+      (effects (font (size 1.27 1.27)) (justify left))
+    )
+    (property "Footprint" "Capacitor_SMD:C_0603_1608Metric" (id 2) (at 103.2002 146.05 0)
+      (effects (font (size 1.27 1.27)) hide)
+    )
+    (property "Datasheet" "~" (id 3) (at 102.235 142.24 0)
+      (effects (font (size 1.27 1.27)) hide)
+    )
+    (pin "1")
+    (pin "2")
+  )
   (symbol (lib_id "Switch:SW_Push_45deg") (at 154.305 82.55 0) (unit 1)
     (in_bom no) (on_board yes) (fields_autoplaced)
-    (property "Reference" "SW8" (id 0) (at 154.305 74.295 0))
+    (property "Reference" "SW7" (id 0) (at 154.305 74.295 0))
     (property "Value" "8" (id 1) (at 154.305 76.835 0))
     (property "Footprint" "Keypad:snap dome" (id 2) (at 154.305 82.55 0)
@@
   (symbol (lib_id "power:GND") (at 53.34 147.955 0) (unit 1)
     (in_bom yes) (on_board yes) (fields_autoplaced)
-    (property "Reference" "#PWR046" (id 0) (at 53.34 154.305 0)
+    (property "Reference" "#PWR042" (id 0) (at 53.34 154.305 0)
       (effects (font (size 1.27 1.27)) hide)
     )
@@
   (symbol (lib_id "Switch:SW_Push_45deg") (at 194.945 97.155 0) (unit 1)
     (in_bom no) (on_board yes) (fields_autoplaced)
-    (property "Reference" "SW17" (id 0) (at 194.945 88.9 0))
+    (property "Reference" "SW16" (id 0) (at 194.945 88.9 0))
     (property "Value" "Call/OK" (id 1) (at 194.945 91.44 0))
     (property "Footprint" "Keypad:snap dome" (id 2) (at 194.945 97.155 0)
@@
   (symbol (lib_id "Switch:SW_Push_45deg") (at 170.18 97.155 0) (unit 1)
     (in_bom no) (on_board yes) (fields_autoplaced)
-    (property "Reference" "SW13" (id 0) (at 170.18 88.9 0))
+    (property "Reference" "SW12" (id 0) (at 170.18 88.9 0))
     (property "Value" "#" (id 1) (at 170.18 91.44 0))
     (property "Footprint" "Keypad:snap dome" (id 2) (at 170.18 97.155 0)
@@
   (symbol (lib_id "Switch:SW_Push_45deg") (at 138.43 82.55 0) (unit 1)
     (in_bom no) (on_board yes) (fields_autoplaced)
-    (property "Reference" "SW4" (id 0) (at 138.43 74.295 0))
+    (property "Reference" "SW3" (id 0) (at 138.43 74.295 0))
     (property "Value" "7" (id 1) (at 138.43 76.835 0))
     (property "Footprint" "Keypad:snap dome" (id 2) (at 138.43 82.55 0)
@@
   (symbol (lib_id "Switch:SW_Push_45deg") (at 170.18 69.215 0) (unit 1)
     (in_bom no) (on_board yes) (fields_autoplaced)
-    (property "Reference" "SW11" (id 0) (at 170.18 60.96 0))
+    (property "Reference" "SW10" (id 0) (at 170.18 60.96 0))
     (property "Value" "6" (id 1) (at 170.18 63.5 0))
     (property "Footprint" "Keypad:snap dome" (id 2) (at 170.18 69.215 0)
@@
   (symbol (lib_id "Switch:SW_Push_45deg") (at 138.43 69.215 0) (unit 1)
     (in_bom no) (on_board yes) (fields_autoplaced)
-    (property "Reference" "SW3" (id 0) (at 138.43 60.96 0))
+    (property "Reference" "SW2" (id 0) (at 138.43 60.96 0))
     (property "Value" "4" (id 1) (at 138.43 63.5 0))
     (property "Footprint" "Keypad:snap dome" (id 2) (at 138.43 69.215 0)
@@
   (symbol (lib_id "Switch:SW_Push_45deg") (at 154.305 69.215 0) (unit 1)
     (in_bom no) (on_board yes) (fields_autoplaced)
-    (property "Reference" "SW7" (id 0) (at 154.305 60.96 0))
+    (property "Reference" "SW6" (id 0) (at 154.305 60.96 0))
     (property "Value" "5" (id 1) (at 154.305 63.5 0))
     (property "Footprint" "Keypad:snap dome" (id 2) (at 154.305 69.215 0)
@@
   (symbol (lib_id "JLCPCB:AW9523BTQR") (at 67.945 132.715 0) (unit 1)
     (in_bom yes) (on_board yes) (fields_autoplaced)
-    (property "Reference" "U5" (id 0) (at 67.945 149.86 0))
+    (property "Reference" "U4" (id 0) (at 67.945 149.86 0))
     (property "Value" "AW9523BTQR" (id 1) (at 67.945 152.4 0))
     (property "Footprint" "lib_fp:QFN-24_EP_4x4_Pitch0.5mm" (id 2) (at 67.945 146.685 0)
@@
     (pin "9")
   )
+  (symbol (lib_id "power:GND") (at 102.235 146.05 0) (unit 1)
+    (in_bom yes) (on_board yes) (fields_autoplaced)
+    (property "Reference" "#PWR046" (id 0) (at 102.235 152.4 0)
+      (effects (font (size 1.27 1.27)) hide)
+    )
+    (property "Value" "GND" (id 1) (at 102.235 150.495 0))
+    (property "Footprint" "" (id 2) (at 102.235 146.05 0)
+      (effects (font (size 1.27 1.27)) hide)
+    )
+    (property "Datasheet" "" (id 3) (at 102.235 146.05 0)
+      (effects (font (size 1.27 1.27)) hide)
+    )
+    (pin "1")
+  )
   (symbol (lib_id "power:+3V3") (at 102.235 138.43 0) (unit 1)
     (in_bom yes) (on_board yes) (fields_autoplaced)
-    (property "Reference" "#PWR049" (id 0) (at 102.235 142.24 0)
+    (property "Reference" "#PWR045" (id 0) (at 102.235 142.24 0)
       (effects (font (size 1.27 1.27)) hide)
     )
@@
   (symbol (lib_id "Switch:SW_Push_45deg") (at 170.18 82.55 0) (unit 1)
     (in_bom no) (on_board yes) (fields_autoplaced)
-    (property "Reference" "SW12" (id 0) (at 170.18 74.295 0))
+    (property "Reference" "SW11" (id 0) (at 170.18 74.295 0))
     (property "Value" "9" (id 1) (at 170.18 76.835 0))
     (property "Footprint" "Keypad:snap dome" (id 2) (at 170.18 82.55 0)
@@
   (symbol (lib_id "Switch:SW_Push_45deg") (at 154.305 55.245 0) (unit 1)
     (in_bom no) (on_board yes) (fields_autoplaced)
-    (property "Reference" "SW6" (id 0) (at 154.305 46.99 0))
+    (property "Reference" "SW5" (id 0) (at 154.305 46.99 0))
     (property "Value" "2" (id 1) (at 154.305 49.53 0))
     (property "Footprint" "Keypad:snap dome" (id 2) (at 154.305 55.245 0)
@@
   (symbol (lib_id "power:GND") (at 83.82 147.955 0) (unit 1)
     (in_bom yes) (on_board yes) (fields_autoplaced)
-    (property "Reference" "#PWR048" (id 0) (at 83.82 154.305 0)
+    (property "Reference" "#PWR044" (id 0) (at 83.82 154.305 0)
       (effects (font (size 1.27 1.27)) hide)
     )
@@
   (symbol (lib_id "Switch:SW_Push_45deg") (at 138.43 55.245 0) (unit 1)
     (in_bom no) (on_board yes) (fields_autoplaced)
-    (property "Reference" "SW2" (id 0) (at 138.43 46.99 0))
+    (property "Reference" "SW1" (id 0) (at 138.43 46.99 0))
     (property "Value" "1" (id 1) (at 138.43 49.53 0))
     (property "Footprint" "Keypad:snap dome" (id 2) (at 138.43 55.245 0)
@@
   (symbol (lib_id "Switch:SW_Push_45deg") (at 154.305 97.155 0) (unit 1)
     (in_bom no) (on_board yes) (fields_autoplaced)
-    (property "Reference" "SW9" (id 0) (at 154.305 88.9 0))
+    (property "Reference" "SW8" (id 0) (at 154.305 88.9 0))
     (property "Value" "0" (id 1) (at 154.305 91.44 0))
     (property "Footprint" "Keypad:snap dome" (id 2) (at 154.305 97.155 0)
@@
   (symbol (lib_id "power:GND") (at 71.755 109.855 0) (unit 1)
     (in_bom yes) (on_board yes) (fields_autoplaced)
-    (property "Reference" "#PWR047" (id 0) (at 71.755 116.205 0)
+    (property "Reference" "#PWR043" (id 0) (at 71.755 116.205 0)
       (effects (font (size 1.27 1.27)) hide)
     )
@@
   (symbol (lib_id "Switch:SW_Push_45deg") (at 194.945 82.55 0) (unit 1)
     (in_bom no) (on_board yes) (fields_autoplaced)
-    (property "Reference" "SW16" (id 0) (at 194.945 74.295 0))
+    (property "Reference" "SW15" (id 0) (at 194.945 74.295 0))
     (property "Value" "Down" (id 1) (at 194.945 76.835 0))
     (property "Footprint" "Keypad:snap dome" (id 2) (at 194.945 82.55 0)
@@
   (symbol (lib_id "Switch:SW_Push_45deg") (at 170.18 55.245 0) (unit 1)
     (in_bom no) (on_board yes) (fields_autoplaced)
-    (property "Reference" "SW10" (id 0) (at 170.18 46.99 0))
+    (property "Reference" "SW9" (id 0) (at 170.18 46.99 0))
     (property "Value" "3" (id 1) (at 170.18 49.53 0))
     (property "Footprint" "Keypad:snap dome" (id 2) (at 170.18 55.245 0)
@@
   (symbol (lib_id "Switch:SW_Push_45deg") (at 194.945 55.245 0) (unit 1)
     (in_bom no) (on_board yes) (fields_autoplaced)
-    (property "Reference" "SW14" (id 0) (at 194.945 46.99 0))
+    (property "Reference" "SW13" (id 0) (at 194.945 46.99 0))
     (property "Value" "End/Back" (id 1) (at 194.945 49.53 0))
     (property "Footprint" "Keypad:snap dome" (id 2) (at 194.945 55.245 0)
@@
   (symbol (lib_id "Switch:SW_Push_45deg") (at 138.43 97.155 0) (unit 1)
     (in_bom no) (on_board yes) (fields_autoplaced)
-    (property "Reference" "SW5" (id 0) (at 138.43 88.9 0))
+    (property "Reference" "SW4" (id 0) (at 138.43 88.9 0))
     (property "Value" "*" (id 1) (at 138.43 91.44 0))
     (property "Footprint" "Keypad:snap dome" (id 2) (at 138.43 97.155 0)

Commit message: First JLCPCB Ship!
Parts:
- C21: renamed from C13; MPN (none) -> C15849
Changed lines of the file:
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@@
   (symbol (lib_id "Device:C") (at 102.235 142.24 0) (unit 1)
     (in_bom yes) (on_board yes) (fields_autoplaced)
-    (property "Reference" "C13" (id 0) (at 105.41 140.9699 0)
+    (property "Reference" "C21" (id 0) (at 105.41 140.9699 0)
       (effects (font (size 1.27 1.27)) (justify left))
     )
@@
     )
     (property "Datasheet" "~" (id 3) (at 102.235 142.24 0)
+      (effects (font (size 1.27 1.27)) hide)
+    )
+    (property "MPN" "C15849" (id 4) (at 102.235 142.24 0)
       (effects (font (size 1.27 1.27)) hide)
     )
@@
   (symbol (lib_id "power:GND") (at 53.34 147.955 0) (unit 1)
     (in_bom yes) (on_board yes) (fields_autoplaced)
-    (property "Reference" "#PWR042" (id 0) (at 53.34 154.305 0)
+    (property "Reference" "#PWR046" (id 0) (at 53.34 154.305 0)
       (effects (font (size 1.27 1.27)) hide)
     )
@@
   (symbol (lib_id "power:GND") (at 102.235 146.05 0) (unit 1)
     (in_bom yes) (on_board yes) (fields_autoplaced)
-    (property "Reference" "#PWR046" (id 0) (at 102.235 152.4 0)
+    (property "Reference" "#PWR050" (id 0) (at 102.235 152.4 0)
       (effects (font (size 1.27 1.27)) hide)
     )
@@
   (symbol (lib_id "power:+3V3") (at 102.235 138.43 0) (unit 1)
     (in_bom yes) (on_board yes) (fields_autoplaced)
-    (property "Reference" "#PWR045" (id 0) (at 102.235 142.24 0)
+    (property "Reference" "#PWR049" (id 0) (at 102.235 142.24 0)
       (effects (font (size 1.27 1.27)) hide)
     )
@@
   (symbol (lib_id "power:GND") (at 83.82 147.955 0) (unit 1)
     (in_bom yes) (on_board yes) (fields_autoplaced)
-    (property "Reference" "#PWR044" (id 0) (at 83.82 154.305 0)
+    (property "Reference" "#PWR048" (id 0) (at 83.82 154.305 0)
       (effects (font (size 1.27 1.27)) hide)
     )
@@
   (symbol (lib_id "power:GND") (at 71.755 109.855 0) (unit 1)
     (in_bom yes) (on_board yes) (fields_autoplaced)
-    (property "Reference" "#PWR043" (id 0) (at 71.755 116.205 0)
-      (effects (font (size 1.27 1.27)) hide)
-    )
+    (property "Reference" "#PWR047" (id 0) (at 71.755 116.205 0)
+      (effects (font (size 1.27 1.27)) hide)
+    )
