File: phone.kicad_pcb (KiCad board)
At the start: 4 copper layers, 37.5 x 130 mm, 124 parts, among them J1 47219-2001, J10 +, J11 -, J2 SWDIO, J3 Display, J4 Bus_PCI_Express_Mini, J5 Battery, J6 USB_C_Receptacle_USB2.0, J7 FH34SRJ-6S-0.5SH(50), J8 FH34SRJ-6S-0.5SH(50), J9 Conn_01x02_Female, SW1 SW_Push, SW10 3, SW11 6, SW12 9, SW13 #, SW14 End/Back, SW15 Up, SW16 Down, SW17 Call/OK, SW2 1, SW3 4, SW4 7, SW5 *, SW6 2, SW7 5, SW8 8, SW9 0, U1 SL2.1S, U2 STM32L432KCUx, U3 BQ24072RGTT, U4 TPS63020DSJR, U5 AW9523BTQR, U6 ALC5672, Y1 X322516MLB4SI

Commit message: Before Shortening
Parts:
- moved R3 2.50 mm to (115.4, 65.8), turned to -90 degrees
- moved R4 1.45 mm to (114.2, 66.5), turned to -90 degrees
Routing:
- net /RST_TFT: track 90.7 -> 84.9 mm
- net /CS_TFT: track 89.9 -> 85.2 mm
- net /BL_TFT: track 92.6 -> 88.1 mm
- net +3V3: track 63.8 -> 60.2 mm
- net /MOSI_TFT: track 98.1 -> 95.0 mm
- net /SDA: track 91.4 -> 94.5 mm
- net /DC_TFT: track 91.4 -> 88.6 mm
- net /MISO_SD: track 34.3 -> 32.1 mm
- net /SCLK_SD: track 28.2 -> 26.0 mm
- net /SCL: track 86.7 -> 88.3 mm
- net /LTE_D+: track 78.5 -> 79.6 mm
- net /keypad/H2: track 75.7 -> 76.7 mm
- net /LTE_D-: track 79.0 -> 79.8 mm
- net /SCLK_TFT: track 97.6 -> 96.8 mm
- net /keypad/H1: track 51.2 -> 51.9 mm
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
Commit message: New Audio
Parts:
- removed C18, C19, C20, C27: 22pF, Capacitor_SMD:C_0402_1005Metric
- removed C28, C31, C49: 4.7uF, Capacitor_SMD:C_0402_1005Metric
- removed C35: 2.2uF, Capacitor_SMD:C_0402_1005Metric
- removed C48, C50: 100nF, Capacitor_SMD:C_0402_1005Metric
- removed the D1 at (135.4, 64.7)
- removed the D2 at (134.3, 64.7)
- removed J10: +, TestPoint:TestPoint_THTPad_2.0x2.0mm_Drill1.0mm
- removed J11: -, TestPoint:TestPoint_THTPad_2.0x2.0mm_Drill1.0mm
- removed J8: FH34SRJ-6S-0.5SH(50), lib_fp:HRS_FH34SRJ-6S-0.5SH(50)
- removed J9: Conn_01x02_Female, Jumper:SolderJumper-2_P1.3mm_Open_Pad1.0x1.5mm
- removed LS2: Earphone, speakerpads:speakerpads
- removed the R5 at (134.3, 66.7)
- removed the R6 at (135.4, 66.7)
- added R18: 10k, Resistor_SMD:R_0402_1005Metric, F.Cu at (52.5, 106.3)
- added R19: 10k, Resistor_SMD:R_0402_1005Metric, F.Cu at (45.3, 114.5)
- added R31: 33, Resistor_SMD:R_0603_1608Metric, F.Cu at (57.0, 101.6)
- added U7: ALC5616-CGT, lib_fp:ALC5616-CGT, F.Cu at (139.2, 120.2)
- added U8: RT9193-18GB, lib_fp:RT9193-18GB, F.Cu at (130.9, 119.0)
- C21, C24: value 22pF -> NC 22pF 6.3V; footprint Capacitor_SMD:C_0402_1005Metric -> Capacitor_SMD:C_0603_1608Metric
- C22, C23, C25: value 4.7uF -> NC 22pF 6.3V; footprint Capacitor_SMD:C_0402_1005Metric -> Capacitor_SMD:C_0603_1608Metric
- C26, C33: value 10uF -> 0.1uF 6.3V
- C29: value 2.2uF -> 4.7uF 6.3V
- C30, C32, C34, C46: value 100nF -> 2.2uF 6.3V
- C36, C38: value 2.2uF -> 2.2uF 6.3V
- C37: value 2.2uF -> 1uF X7R
- C39, C40: value 1uF -> 0.1uF 6.3V
- C41: value 680pF -> 4.7uF 6.3V
- C42: value 680pF -> 2.2uF 6.3V
- C43: value 680pF -> 0.1uF 6.3V
- C44: value 680pF -> 22nF
- C45: value 2.2uF -> 0.1uF 6.3V
- C47: value 4.7uF -> 1uF X7R
- D1: renamed from D3; footprint LED_SMD:LED_0402_1005Metric -> LED_SMD:LED_0603_1608Metric
- D2: renamed from D4; value LED -> GREEN LED; footprint LED_SMD:LED_0402_1005Metric -> LED_SMD:LED_0603_1608Metric
- D3: renamed from D5; value LED -> YELLOW LED; footprint LED_SMD:LED_0402_1005Metric -> LED_SMD:LED_0603_1608Metric
- R10: renamed from R12; value 1.5k -> 68
- R20, R21: value 0 -> 20k; footprint Resistor_SMD:R_0402_1005Metric -> Resistor_SMD:R_0603_1608Metric
- R22, R23: value 22 -> 20k; footprint Resistor_SMD:R_0402_1005Metric -> Resistor_SMD:R_0603_1608Metric
- R24: value 1k -> 20k; footprint Resistor_SMD:R_0402_1005Metric -> Resistor_SMD:R_0603_1608Metric
- R25: value 1k -> 47; footprint Resistor_SMD:R_0402_1005Metric -> Resistor_SMD:R_0603_1608Metric
- R26, R27: value 10k -> 0; footprint Resistor_SMD:R_0402_1005Metric -> Resistor_SMD:R_0603_1608Metric
- R28, R29: value 1k -> 22; footprint Resistor_SMD:R_0402_1005Metric -> Resistor_SMD:R_0603_1608Metric
- R30: value 0 -> 33; footprint Resistor_SMD:R_0402_1005Metric -> Resistor_SMD:R_0603_1608Metric
- R5: renamed from R7; value 470 -> 68
- R9: renamed from R11; value 1.5k -> 1
- U6: value ALC5672 -> LM4889MMX/NOPB; footprint lib_fp:ALC5672-VB-CGT_QFN-48_EP_6x6_Pitch0.4mm -> lib_fp:LM4889MMX&slash_NOPB
- moved C47 124.7 mm to (45.2, 118.4)
- moved C26 123.7 mm to (41.2, 120.3)
- moved C40 121.7 mm to (48.1, 115.9)
- moved R21 121.1 mm to (37.8, 115.5), turned to 0 degrees
- moved R28 118.9 mm to (44.3, 112.2)
- moved R22 118.1 mm to (48.4, 109.7), turned to 0 degrees
- moved C43 117.6 mm to (45.2, 116.5), turned to 0 degrees
- moved C38 116.7 mm to (47.8, 112.0), turned to 0 degrees
- moved R26 115.5 mm to (41.8, 118.0)
- moved C37 113.3 mm to (51.8, 108.8), turned to 0 degrees
- moved R23 112.3 mm to (49.0, 106.6), turned to 0 degrees
- moved C41 112.1 mm to (56.5, 103.8), turned to 0 degrees
- moved R29 109.1 mm to (49.0, 101.6)
- moved C33 108.2 mm to (48.1, 113.9), turned to 0 degrees
- moved R27 106.9 mm to (44.3, 109.7), turned to 0 degrees
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- renumbered R13 to R11, R14 to R12, R15 to R13, R16 to R14, R17 to R15, R18 to R16, R19 to R17, R8 to R6, R9 to R7, R10 to R8
Connections:
- C21 pad 1: GND -> /PCM_DOUT
- C21 pad 2: Net-(C21-Pad2) -> GND
- C22 pad 1: GNDA -> /PCM_CLK
- C22 pad 2: Net-(C22-Pad2) -> GND
- C23 pad 1: Net-(C23-Pad1) -> GND
- C23 pad 2: GNDA -> /PCM_DIN
- C24 pad 2: Net-(C24-Pad2) -> /PCM_SYNC
- C25 pad 1: GNDA -> GND
- C25 pad 2: Net-(C25-Pad2) -> /audio/MCLK
- C26 pad 1: Net-(C26-Pad1) -> +1V8
- C29 pad 1: GND -> GNDA
- C29 pad 2: +3V3 -> Net-(C29-Pad2)
- C30 pad 1: GND -> Net-(C30-Pad1)
- C30 pad 2: +3V3 -> Net-(C30-Pad2)
- C32 pad 1: GND -> Net-(C32-Pad1)
- C32 pad 2: Net-(C31-Pad2) -> Net-(C32-Pad2)
- C33 pad 1: +3V3 -> +1V8
- C33 pad 2: GND -> GNDA
- C34 pad 1: GND -> GNDA
- C34 pad 2: +3V3 -> Net-(C34-Pad2)
- C36 pad 1: Net-(C36-Pad1) -> GNDA
- C37 pad 1: GNDA -> GND
- C37 pad 2: Net-(C37-Pad2) -> +3V3
- C39 pad 1: Net-(C39-Pad1) -> +3V3
- C39 pad 2: Net-(C39-Pad2) -> GNDA
- C41 pad 1: Net-(C41-Pad1) -> GNDA
- C41 pad 2: GND -> +3V3
- C43 pad 1: GND -> Net-(C43-Pad1)
- C43 pad 2: GND -> Net-(C43-Pad2)
- C44 pad 1: Net-(C44-Pad1) -> GND
- C44 pad 2: GND -> Net-(C44-Pad2)
- C45 pad 2: DBVDD -> +1V8
- C46 pad 1: GND -> +1V8
- C46 pad 2: DBVDD -> GND
- C47 pad 1: /audio/CPVDD -> GND
- C47 pad 2: GNDA -> +1V8
- D1 pad 1: GND -> Net-(D1-Pad1)
- J4 pad 30: /audio/SCL_CODEC -> /audio/SCL
- J4 pad 32: /audio/SDA_CODEC -> /audio/SDA
- J4 pad 42: Net-(J4-Pad42) -> Net-(D1-Pad1)
- J4 pad 44: Net-(J4-Pad44) -> unconnected-(J4-Pad44)
- J4 pad 46: Net-(J4-Pad46) -> unconnected-(J4-Pad46)
- R20 pad 1: Net-(C22-Pad2) -> Net-(R20-Pad1)
- R20 pad 2: Net-(R20-Pad2) -> Net-(C19-Pad1)
- R21 pad 1: Net-(C23-Pad1) -> Net-(R21-Pad1)
- R21 pad 2: Net-(R21-Pad2) -> Net-(C20-Pad1)
- R22 pad 1: Net-(R22-Pad1) -> Net-(C18-Pad1)
- R22 pad 2: Net-(C39-Pad1) -> Net-(R20-Pad1)
- R23 pad 1: Net-(R23-Pad1) -> /audio/AMP_OFF
- R23 pad 2: Net-(C40-Pad1) -> +3V3
- R24 pad 1: Net-(R24-Pad1) -> Net-(R21-Pad1)
- R24 pad 2: Net-(C44-Pad1) -> Net-(LS1-Pad1)
- R25 pad 1: Net-(R25-Pad1) -> +1V8
- R25 pad 2: Net-(C44-Pad1) -> Net-(C28-Pad1)
- R26 pad 1: /audio/SDA_CODEC -> GND
- R26 pad 2: DBVDD -> GNDA
- R27 pad 1: /audio/SCL_CODEC -> unconnected-(R27-Pad1)
- R27 pad 2: DBVDD -> Net-(R27-Pad2)
- R28 pad 1: Net-(R28-Pad1) -> GNDA
- R28 pad 2: Net-(C41-Pad1) -> Net-(C40-Pad2)
- R29 pad 1: Net-(R29-Pad1) -> GNDA
- R29 pad 2: Net-(C41-Pad1) -> Net-(C43-Pad1)
- R30 pad 1: GND -> unconnected-(R30-Pad1)
- R30 pad 2: GNDA -> Net-(C43-Pad2)
- R5 pad 1: Net-(J4-Pad42) -> +3V3
- U3 pad : GNDPWR -> (no net)
- U4 pad 16: GNDPWR -> (no net)
- U4 pad 17: GNDPWR -> (no net)
- U4 pad 18: GNDPWR -> (no net)
- U4 pad 19: GNDPWR -> (no net)
- U4 pad 20: GNDPWR -> (no net)
- U4 pad 21: GNDPWR -> (no net)
- U4 pad 22: GNDPWR -> (no net)
- U4 pad 23: GNDPWR -> (no net)
- U4 pad 24: GNDPWR -> (no net)
- U4 pad 25: GNDPWR -> (no net)
- U4 pad 26: GNDPWR -> (no net)
- U4 pad 27: GNDPWR -> (no net)
- U4 pad 28: GNDPWR -> (no net)
- U4 pad 29: GNDPWR -> (no net)
- U4 pad 30: GNDPWR -> (no net)
- U6 pad 1: Net-(R24-Pad1) -> /audio/AMP_OFF
- U6 pad 2: DBVDD -> Net-(C18-Pad1)
- U6 pad 3: Net-(C31-Pad2) -> Net-(R20-Pad1)
- U6 pad 4: /audio/OUT2+ -> Net-(R21-Pad1)
- U6 pad 5: /audio/OUT2- -> Net-(LS1-Pad1)
- U6 pad 6: /audio/AVDD -> +3V3
- U6 pad 7: Net-(C28-Pad1) -> GND
- U6 pad 8: Net-(C25-Pad2) -> Net-(LS1-Pad2)
Routing:
- net DBVDD: track 176.3 -> 0.00 mm, vias 4 -> 0
- net /audio/OUT1-: track 123.6 -> 0.00 mm
- net /audio/OUT1+: track 123.1 -> 0.00 mm
- net /audio/OUT2+: track 124.1 -> 6.30 mm, vias 2 -> 1
- net /audio/OUT2-: track 123.5 -> 7.44 mm, vias 2 -> 1
- net GND: track 175.2 -> 107.7 mm, vias 52 -> 36
- net /audio/SDA_CODEC: track 62.1 -> 0.00 mm, vias 2 -> 0
- net /audio/SCL_CODEC: track 61.9 -> 0.00 mm, vias 2 -> 0
- net /PCM_DIN: track 82.2 -> 37.7 mm
- net /PCM_DOUT: track 81.1 -> 37.1 mm, vias 2 -> 0
- net /PCM_CLK: track 76.7 -> 36.8 mm, vias 2 -> 0
- net /PCM_SYNC: track 76.7 -> 37.0 mm
- net GNDA: track 30.8 -> 0.00 mm, vias 5 -> 0
- net /audio/SDA: track 0.00 -> 28.6 mm, vias 0 -> 1
- net /audio/SCL: track 0.00 -> 28.3 mm, vias 0 -> 1
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- removed copper zone on F.Cu, net GNDA
- removed copper zone on In2.Cu, net GNDA
Other:
- board size 37.5 x 130 mm -> 37.5 x 120 mm

Commit message: Getting There
Need to move keyboard down and finish routing to audio, then we're there!
Parts:
- removed the C1 at (115.5, 141.8)
- removed the C2 at (110.0, 141.8)
- removed the C4 at (110.8, 138.2)
- removed the C5 at (109.5, 137.0)
- removed the C6 at (115.7, 134.0)
- removed the SW1 at (121.5, 118.7)
- removed the U1 at (112.3, 134.1)
- removed the U6 at (126.5, 35.8)
- removed Y1: X322516MLB4SI, lib_fp:OSC_X322516MLB4SI
- added C13: 1uF, Capacitor_SMD:C_0603_1608Metric, F.Cu at (122.5, 86.2)
- added C14: 1uF 6.3V, Capacitor_SMD:C_0402_1005Metric, F.Cu at (121.2, 34.5)
- added C15: 100nF 6.3V, Capacitor_SMD:C_0402_1005Metric, F.Cu at (117.2, 37.8)
- added C16: 100nF 6.3V, Capacitor_SMD:C_0402_1005Metric, F.Cu at (119.0, 41.0)
- added C23: 4.7uF 6.3V, Capacitor_SMD:C_0402_1005Metric, F.Cu at (127.0, 109.7)
- added C24: 1uF 6.3V, Capacitor_SMD:C_0402_1005Metric, F.Cu at (129.0, 38.0)
- added C25: 4.7uF 6.3V, Capacitor_SMD:C_0402_1005Metric, F.Cu at (127.0, 111.7)
- added C31: 4.7uF 6.3V, Capacitor_SMD:C_0402_1005Metric, F.Cu at (122.8, 117.2)
- added JP1: SolderJumper_2_Open, Jumper:SolderJumper-2_P1.3mm_Open_Pad1.0x1.5mm, F.Cu at (118.9, 119.6)
- added LS1: Earphone, Connector_PinHeader_1.27mm:PinHeader_1x02_P1.27mm_Vertical, F.Cu at (131.2, 38.8)
- added U5: LM4889MM, lib_fp:LM4889MM, F.Cu at (125.0, 38.0)
- C22: renamed from C26; value 0.1uF 6.3V -> 100nF 6.3V
- C29: renamed from C33; value 0.1uF 6.3V -> 100nF 6.3V
- C3: renamed from C8; value 1uF X5R -> 1uF X7R
- C35: renamed from C39; value 0.1uF 6.3V -> 100nF 6.3V
- C36: renamed from C40; value 0.1uF 6.3V -> 100nF 6.3V
- C39: renamed from C43; value 0.1uF 6.3V -> 100nF 6.3V
- C41: renamed from C45; value 0.1uF 6.3V -> 100nF 6.3V
- R12, R13: footprint Resistor_SMD:R_0402_1005Metric -> Resistor_SMD:R_0603_1608Metric
- moved R26 127.7 mm to (167.2, 142.0)
- moved R20 111.7 mm to (120.5, 40.5), turned to -90 degrees
- moved R22 104.5 mm to (147.3, 91.7)
- moved R23 103.3 mm to (122.8, 34.2), turned to 90 degrees
- moved R21 102.3 mm to (120.5, 37.2), turned to -90 degrees
- moved R18 95.7 mm to (147.2, 93.0)
- moved R24 93.9 mm to (125.2, 41.5), turned to 90 degrees
- moved C22 87.7 mm to (128.2, 109.7), turned to 90 degrees
- moved C43 87.0 mm to (132.2, 117.0), turned to -90 degrees
- moved C33 86.8 mm to (138.2, 116.3), turned to -90 degrees
- moved R27 85.4 mm to (129.8, 111.0), turned to -90 degrees
- moved C38 81.2 mm to (132.2, 112.8), turned to 90 degrees
- moved R28 81.2 mm to (124.2, 126.5), turned to -90 degrees
- moved C40 80.6 mm to (132.2, 115.0), turned to 90 degrees
- moved C39 79.1 mm to (124.0, 123.8), turned to -90 degrees
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- renumbered C3 to C1, C15 to C10, C16 to C11, C17 to C12, C21 to C17, C22 to C18, C23 to C19, C7 to C2, C24 to C20, C25 to C21, C29 to C26, C30 to C27, C32 to C28, C34 to C30, C36 to C32, C37 to C33, C38 to C34, C41 to C37, C42 to C38, C9 to C4, C44 to C40, C46 to C42, C47 to C43, C10 to C5, C11 to C6, C12 to C7, C13 to C8, C14 to C9, JP1 to JP2, R20 to R19, R21 to R20, R22 to R21, R19 to R22, SW2 to SW1, SW11 to SW10, SW12 to SW11, SW13 to SW12, SW14 to SW13, SW15 to SW14, SW16 to SW15, SW17 to SW16, SW3 to SW2, SW4 to SW3, SW5 to SW4, SW6 to SW5, SW7 to SW6, SW8 to SW7, SW9 to SW8, SW10 to SW9, U2 to U1, U3 to U2, U4 to U3, U5 to U4, U7 to U6, U8 to U7
Connections:
- J4 pad 11: unconnected-(J4-Pad11) -> /UART_RX
- J4 pad 13: unconnected-(J4-Pad13) -> /UART_TX
- J4 pad 36: /LTE_D- -> unconnected-(J4-Pad36)
- J4 pad 38: /LTE_D+ -> unconnected-(J4-Pad38)
- J6 pad A6: /USB/USB_D+ -> /MCU_D-
- J6 pad A7: /USB/USB_D- -> /MCU_D+
- J6 pad B6: /USB/USB_D+ -> /MCU_D-
- J6 pad B7: /USB/USB_D- -> /MCU_D+
- U1 pad 29: unconnected-(U2-Pad29) -> /UART_TX
- U1 pad 30: /PG_PWR -> /UART_RX
Routing:
- net /LTE_D-: track 79.8 -> 0.00 mm, vias 2 -> 0
- net /LTE_D+: track 79.6 -> 0.00 mm, vias 2 -> 0
- net /PCM_DIN: track 37.7 -> 0.00 mm
- net /PCM_DOUT: track 37.1 -> 0.00 mm
- net /PCM_SYNC: track 37.0 -> 0.00 mm
- net /PCM_CLK: track 36.8 -> 0.00 mm
- net /SDA: track 94.5 -> 60.1 mm
- net /audio/SDA: track 28.6 -> 0.00 mm, vias 1 -> 0
- net /audio/SCL: track 28.3 -> 0.00 mm, vias 1 -> 0
- net /SCL: track 88.3 -> 62.1 mm, vias 4 -> 2
- net /MCU_D-: track 7.30 -> 30.9 mm, vias 0 -> 2
- net /MCU_D+: track 7.00 -> 30.3 mm
- net /PG_BATT: track 32.5 -> 9.97 mm, vias 3 -> 0
- net +5V: track 21.3 -> 0.00 mm, vias 2 -> 0
- net /USB/USB_D-: track 19.2 -> 0.00 mm, vias 2 -> 0
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- added copper zone on B.Cu, net GNDPWR

Commit message: First JLCPCB Ship!
Parts:
- removed R26: 0, Resistor_SMD:R_0603_1608Metric
- added NT1: NetTie_2, NetTie:NetTie-2_SMD_Pad0.5mm, F.Cu at (120.2, 141.2)
- C14, C15, C16, C24: footprint Capacitor_SMD:C_0402_1005Metric -> Capacitor_SMD:C_0603_1608Metric
- J3: moved to F.Cu
- moved R19 25.4 mm to (131.6, 59.2)
- moved R23 25.4 mm to (136.2, 55.8), turned to -90 degrees
- moved D1 24.9 mm to (131.6, 81.4)
- moved C15 24.7 mm to (129.6, 59.2)
- moved R20 24.7 mm to (131.6, 62.6)
- moved C14 24.7 mm to (133.8, 55.8)
- moved R5 24.4 mm to (130.0, 81.0), turned to -90 degrees
- moved R22 24.3 mm to (135.6, 113.0), turned to 90 degrees
- moved C24 24.2 mm to (140.1, 59.5)
- moved U5 24.2 mm to (136.1, 59.5)
- moved LS1 24.1 mm to (142.5, 60.1)
- moved C16 24.0 mm to (129.6, 62.6), turned to 90 degrees
- moved R18 23.9 mm to (134.1, 113.0), turned to 90 degrees
- moved R24 23.3 mm to (133.8, 63.2), turned to -90 degrees
- moved R21 21.6 mm to (131.6, 55.8)
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Connections:
- C22 pad 1: +1V8 -> DBVDD
- C23 pad 1: +1V8 -> DBVDD
- C29 pad 1: +1V8 -> DBVDD
- C31 pad 1: +1V8 -> DBVDD
- C41 pad 2: +1V8 -> DBVDD
- C42 pad 1: +1V8 -> DBVDD
- C43 pad 2: +1V8 -> DBVDD
- R25 pad 1: +1V8 -> DBVDD
- U6 pad 15: +1V8 -> DBVDD
- U6 pad 29: +1V8 -> DBVDD
- U6 pad 6: +1V8 -> DBVDD
- U7 pad 5: +1V8 -> DBVDD
Routing:
- net /audio/SCL: track 0.00 -> 84.9 mm, vias 0 -> 2
- net /audio/SDA: track 0.00 -> 84.0 mm, vias 0 -> 2
- net DBVDD: track 0.00 -> 71.8 mm, vias 0 -> 7
- net /audio/IN+: track 0.00 -> 65.1 mm, vias 0 -> 2
- net /audio/IN-: track 0.00 -> 64.8 mm, vias 0 -> 2
- net /UART_RX: track 1.99 -> 64.9 mm, vias 1 -> 2
- net /PCM_DIN: track 0.00 -> 62.4 mm
- net /PCM_DOUT: track 0.00 -> 61.4 mm
- net /PCM_SYNC: track 0.00 -> 60.7 mm, vias 0 -> 2
- net /PCM_CLK: track 0.00 -> 59.2 mm
- net /UART_TX: track 10.1 -> 60.7 mm, vias 1 -> 2
- net GNDA: track 18.2 -> 55.8 mm, vias 3 -> 9
- net GND: track 100.8 -> 135.1 mm, vias 34 -> 41
- net /audio/MCLK: track 0.00 -> 17.3 mm
- net /audio/OUT2+: track 24.7 -> 40.5 mm
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Other:
- board size 37.5 x 120 mm -> 37.5 x 98.8 mm
