File: phone.kicad_sch (KiCad schematic)
At the start: 26 parts, among them J1 47219-2001, J2 SWDIO, J3 Display, J4 Bus_PCI_Express_Mini, SW1 SW_Push, U1 SL2.1S, U2 STM32L432KCUx, Y1 X322516MLB4SI

Commit message: Before Shortening
Parts:
- removed D1, D2: LED, LED_SMD:LED_0402_1005Metric, symbol Device:LED
- removed R5, R6: 470, Resistor_SMD:R_0402_1005Metric, symbol RobotProtos:RSMALL
- D3: footprint LED_SMD:LED_0402_1005Metric -> LED_SMD:LED_0603_1608Metric; MPN (none) -> C2286
- R7: value 470 -> 68
Connections:
- net +3V3: now also R7.1
- net GND: no longer D3.1 (K)
- net at J4.42 (~{LED_WWAN}): now also D3.1 (K); no longer R7.1
Other:
- moved on the sheet: D3, R7

Commit message: New Audio
Parts:
- renumbered D3 to D1, R7 to R5
Other:
- sheet audio ports: added 1V8_EN, AMP_OFF, MCLK; removed none

Commit message: Getting There
Need to move keyboard down and finish routing to audio, then we're there!
Parts:
- removed C1, C2: 33pF, Capacitor_SMD:C_0402_1005Metric, symbol Device:C
- removed C4, C5: 10uF, Capacitor_SMD:C_0402_1005Metric, symbol Device:C
- removed C6: 100nF, Capacitor_SMD:C_0402_1005Metric, symbol Device:C
- removed SW1: SW_Push, Button_Switch_SMD:SW_SPST_TL3342, symbol Switch:SW_Push
- removed U1: SL2.1S, lib_fp:SL2.1S, symbol JLCPCB:SL2.1S
- removed Y1: X322516MLB4SI, lib_fp:OSC_X322516MLB4SI, symbol JLCPCB:X322516MLB4SI
- added JP1: SolderJumper_2_Open, Jumper:SolderJumper-2_P1.3mm_Open_Pad1.0x1.5mm, symbol Jumper:SolderJumper_2_Open
- renumbered C3 to C1, C7 to C2, JP1 to JP2, U2 to U1
Connections:
- net GND: now also JP1.1 (A)
- net PG_PWR: no longer U1.30 (PB7)
- net UART_RX: now reaches J4.11 (REFCLK-)
- net UART_RX: now also U1.30 (PB7)
- net UART_TX: now reaches J4.13 (REFCLK+)
- net UART_TX: now also U1.29 (PB6)
- net at C2.2, U1.4 (NRST): now also JP1.2 (B)
- net LTE_D+: no longer names the net of J4.38 (USB_D+)
- net LTE_D-: no longer names the net of J4.36 (USB_D-)
- no-connect marks 36 -> 31

Commit message: First JLCPCB Ship!
Parts:
- C1, C2: MPN (none) -> C1525
- J3: now left out of the parts list
- R1, R2: MPN (none) -> C25744
- R3, R4: MPN (none) -> C25900
